File: Delta MUX.kicad_sch (KiCad schematic)
At the start: 24 parts, among them U3 OPA376xxDBV, U5 TMUX1308, U6 OPA376xxDBV, U7 TMUX1308

Commit message: 10.04.2026
Parts:
- removed U3, U6: OPA376xxDBV, Package_TO_SOT_SMD:SOT-23-5, symbol Amplifier_Operational:OPA376xxDBV
- added R20, R21, R22, R23, R24, R25, R26, R27, R28, R29, R30, R31, R32, R33, R34, R35: R_Small, symbol Device:R_Small
- added U3, U8: OPA365xxDBV, Package_TO_SOT_SMD:SOT-23-5, symbol Amplifier_Operational:OPA365xxDBV
- R11, R12, R13, R15, R5, R6, R7, R9: value 220R -> 330R
- R14, R8: value 22k -> 33k
Connections:
- net +3.3VA: now also U3.5 (V+), U8.5 (V+)
- net COL0: now also R23.1
- net COL1: now also R27.1
- net COL10: now also R30.1
- net COL11: now also R34.1
- net COL12: now also R29.1
- net COL13: now also R33.1
- net COL14: now also R28.1
- net COL15: now also R32.1
- net COL2: now also R22.1
- net COL3: now also R26.1
- net COL4: now also R21.1
- net COL5: now also R25.1
- net COL6: now also R20.1
- net COL7: now also R24.1
- net COL8: now also R31.1
- net COL9: now also R35.1
- net GND: now also R20.2, R21.2, R22.2, R23.2, R24.2, R25.2, R26.2, R27.2, R28.2, R29.2, R30.2, R31.2, R32.2, R33.2, R34.2, R35.2, U3.2 (V-), U8.2 (V-)
- net at R14.1, R15.2: now also U8.4 (-)
- net at R13.1, R14.2: now also U8.1
- net at R8.1, R9.2: now also U3.4 (-)
- net at C22.1, R11.1, R12.2: now also U8.3 (+)
- net at R7.1, R8.2: now also U3.1
- net at C11.1, R5.1, R6.2: now also U3.3 (+)

Commit message: 12.04.2026
Parts:
- removed C12, C23: 470pF, Capacitor_SMD:C_0603_1608Metric, symbol Device:C_Small
- removed R11, R13, R5, R7: 330R, Resistor_SMD:R_0603_1608Metric, symbol Device:R_Small
Connections:
- net ADC0: now also R8.2, U3.1
- net ADC1: now also R14.2, U8.1
- net DISCHARGE0: now also C11.1, R6.2, U3.3 (+)
- net DISCHARGE1: now also C22.1, R12.2, U8.3 (+)
