File: Delta.kicad_sch (KiCad schematic)
At the start: 0 parts

Commit message: 08.04.2026
Parts:
- added C1, C10, C16: 1uF, Capacitor_SMD:C_0603_1608Metric, symbol Device:C_Small
- added C11, C12, C13, C4, C5, C6, C7, C8, C9: 100nF, Capacitor_SMD:C_0402_1005Metric, symbol Device:C_Small
- added C14, C15: 470pF, Capacitor_SMD:C_0603_1608Metric, symbol Device:C_Small
- added C17, C2, C3: 10uF, Capacitor_SMD:C_0805_2012Metric, symbol Device:C_Small
- added F1: 500mA, Fuse:Fuse_0603_1608Metric, symbol Device:Fuse_Small
- added J1: USB_C_Receptacle_USB2.0_16P, Connector_USB:USB_C_Receptacle_G-Switch_GT-USB-7010ASV, symbol Connector:USB_C_Receptacle_USB2.0_16P
- added J8: Conn_ARM_SWD_TagConnect_TC2030-NL, PCM_marbastlib-various:CON_TC2030_outlined, symbol Connector:Conn_ARM_SWD_TagConnect_TC2030-NL
- added P1: PLACEHOLDER 0805-1206, Resistor_SMD:R_0805_2012Metric_Pad1.20x1.40mm_HandSolder, symbol Device:R_Small
- added R1, R15: 22k, Resistor_SMD:R_0603_1608Metric, symbol Device:R_Small
- added R10, R11, R12, R13, R14, R16, R5, R7, R9: 220R, Resistor_SMD:R_0603_1608Metric, symbol Device:R_Small
- added R2, R3: 5.1k, Resistor_SMD:R_0402_1005Metric, symbol Device:R_Small
- added R4: 22R, Resistor_SMD:R_0603_1608Metric, symbol Device:R_Small
- added SW_BOOT1: SW_Push, TestPoint:TestPoint_2Pads_Pitch2.54mm_Drill0.8mm, symbol Switch:SW_Push
- added SW_BOOT2: SW_Push, Button_Switch_SMD:SW_SPST_B3U-1000P, symbol Switch:SW_Push
- added U1: USBLC6-2P6, Package_TO_SOT_SMD:SOT-563, symbol Power_Protection:USBLC6-2P6
- added U2: AT32F405KCU7-4, Package_DFN_QFN:QFN-32-1EP_4x4mm_P0.4mm_EP2.65x2.65mm_ThermalVias, symbol PCM_marbastlib-various:AT32F405KCU7-4
- added U3: STM32G431CBTx, Package_QFP:LQFP-48_7x7mm_P0.5mm, symbol MCU_ST_STM32G4:STM32G431CBTx
- added U5: OPA376xxDBV, Package_TO_SOT_SMD:SOT-23-5, symbol Amplifier_Operational:OPA376xxDBV
- added U6: TPS7A2033, Package_TO_SOT_SMD:SOT-23-5, symbol Kicad symbols:TPS7A20xxx SOT-23-5
Connections:
- new net: J1.A5 (CC1), R2.1
- new net: R14.1, U3.29 (PB15)
- new net: P1.1, R15.1, R16.2, U5.4 (-)
- new net: R5.1, U3.12 (PA4)
- new net: J1.B5 (CC2), R3.1
- new net: P1.2, R13.1, R15.2, U5.1
- new net: C14.1, R11.1, R12.2, U5.3 (+)
- new net: R7.1, U3.30 (PA8)
- new net: R9.1, U3.31 (PA9)
- new net: R10.1, U3.32 (PA10)
- new net: U2.1 (VDD), U2.20 (VDD)
- new net +3.3V: C1.2, C17.1, C3.1, C4.2, C5.2, C6.2, C7.1, J8.1 (VCC), R4.1, SW_BOOT1.1, SW_BOOT2.1, U3.1 (VBAT), U3.24 (VDD), U3.36 (VDD), U3.48 (VDD), U6.5 (OUT)
- new net +3.3VA: C10.2, C12.2, C13.1, C2.2, C8.2, C9.2, R4.2, U3.20 (VREF+), U3.21 (VDDA), U5.5 (V+)
- new net +5V: C16.1, F1.2, U6.1 (IN), U6.3 (EN)
- new net 5V_IN: F1.1, J1.A4 (VBUS), J1.A9 (VBUS), J1.B4 (VBUS), J1.B9 (VBUS), U1.5 (VBUS)
- new net ADC: C15.1, R13.2, U3.18 (PB2)
- new net BOOT0: R1.1, SW_BOOT1.2, SW_BOOT2.2, U3.43 (PB6)
- new net COM: R12.1
- new net D+: U1.1 (I/O1), U3.34 (PA12)
- new net D-: U1.3 (I/O2), U3.33 (PA11)
- new net DISCHARGE: R11.2, U3.13 (PA5)
- new net DN_IN: J1.A7 (D-), J1.B7 (D-), U1.4 (I/O2)
- new net DP_IN: J1.A6 (D+), J1.B6 (D+), U1.6 (I/O1)
- new net GND: C1.1, C10.1, C11.2, C12.1, C13.2, C14.2, C15.2, C16.2, C17.2, C2.1, C3.2, C4.1, C5.1, C6.1, C7.2, C8.1, C9.1, J1.A1 (GND), J1.A12 (GND), J1.B1 (GND), J1.B12 (GND), J1.S1 (SHIELD), J8.5 (GND), J8.6 (SWO), R1.2, R16.1, R2.2, R3.2, U1.2 (GND), U3.19 (VSSA), U3.23 (VSS), U3.35 (VSS), U3.47 (VSS), U5.2 (V-), U6.2 (GND)
- new net MUX_EN0: U3.42 (PB5)
- new net MUX_EN1: U3.44 (PB7)
- new net MUX_S0: U3.39 (PA15)
- new net MUX_S1: U3.40 (PB3)
- new net MUX_S2: U3.41 (PB4)
- new net RESET: C11.1, J8.3 (~{RESET}), U3.7 (PG10)
- new net ROW0: R10.2
- new net ROW1: R9.2
- new net ROW2: R7.2
- new net ROW3: R14.2
- new net ROW4: R5.2
- new net SWCLK: J8.4 (SWCLK), U3.38 (PA14)
- new net SWDIO: J8.2 (SWDIO), U3.37 (PA13)
- no-connect marks 0 -> 23
Other:
- note added: "ADC: 5,6,8-18"
- note added: "External OPAMP x50 + Internal x2"
- note added: "No Osc"
- note added: "ST rec: 10n + 1u"

Commit message: 09.04.2026
Parts:
- removed C11, C12, C13: 100nF, Capacitor_SMD:C_0402_1005Metric, symbol Device:C_Small
- removed C14, C15: 470pF, Capacitor_SMD:C_0603_1608Metric, symbol Device:C_Small
- removed P1: PLACEHOLDER 0805-1206, Resistor_SMD:R_0805_2012Metric_Pad1.20x1.40mm_HandSolder, symbol Device:R_Small
- removed R10, R11, R12, R13, R14, R16, R5, R7, R9: 220R, Resistor_SMD:R_0603_1608Metric, symbol Device:R_Small
- removed R15: 22k, Resistor_SMD:R_0603_1608Metric, symbol Device:R_Small
- removed U2: AT32F405KCU7-4, Package_DFN_QFN:QFN-32-1EP_4x4mm_P0.4mm_EP2.65x2.65mm_ThermalVias, symbol PCM_marbastlib-various:AT32F405KCU7-4
- removed U3: STM32G431CBTx, Package_QFP:LQFP-48_7x7mm_P0.5mm, symbol MCU_ST_STM32G4:STM32G431CBTx
- removed U5: OPA376xxDBV, Package_TO_SOT_SMD:SOT-23-5, symbol Amplifier_Operational:OPA376xxDBV
- added C1: 100nF, symbol Device:C_Small
- added R4: 12k 1%, symbol Device:R_Small
- added SW_RST1: SW_Push, TestPoint:TestPoint_2Pads_Pitch2.54mm_Drill0.8mm, symbol Switch:SW_Push
- added SW_RST2: SW_Push, Button_Switch_SMD:SW_SPST_B3U-1000P, symbol Switch:SW_Push
- added U2: AT32F405CCT, Package_QFP:LQFP-48_7x7mm_P0.5mm, symbol Kicad symbols:AT32F405CCT
- added U8: STM32G473CCTx, Package_QFP:LQFP-48_7x7mm_P0.5mm, symbol MCU_ST_STM32G4:STM32G473CCTx
- added U9: STM32G473RCTx, Package_QFP:LQFP-64_10x10mm_P0.5mm, symbol MCU_ST_STM32G4:STM32G473RCTx
- renumbered C16 to C13, C17 to C14, C1 to C15, C2 to C16, C3 to C2, C4 to C3, C5 to C4, C6 to C5, C7 to C6, C8 to C7, C9 to C8, C10 to C9, J8 to J2, R4 to R10, U6 to U4
Connections:
- net +3.3V: now also U2.1 (VBAT), U2.19 (VDD), U2.28 (VDD), U2.48 (VDD)
- net +3.3VA: now also U2.9 (VDDA)
- net BOOT0: now also U2.44 (PF11/BOOT0)
- net D+: now also U2.27 (OTGHS_D+)
- net D-: now also U2.26 (OTGHS_D-)
- net GND: now also C1.2, R4.1, SW_RST1.2, SW_RST2.2, U2.47 (VSS), U2.8 (VSSA); no longer J2.6 (SWO)
- net RESET: now also C1.1, SW_RST1.1, SW_RST2.1, U2.7 (NRST)
- net SWCLK: now also U2.37 (PA14)
- net SWDIO: now also U2.34 (PA13)
- new net: U8.23 (VSS), U8.35 (VSS), U8.47 (VSS)
- new net: R4.2, U2.25 (OTGHS1_R)
- new net: U9.15 (VSS), U9.31 (VSS), U9.47 (VSS), U9.63 (VSS)
- new net SWO: J2.6 (SWO), U2.39 (PB3)
- no-connect marks 23 -> 3
Other:
- added sheet Delta MATRIX (Delta Matrix.kicad_sch)
- added sheet Delta MUX (Delta MUX.kicad_sch)
- note added: "ADC 10-19"
- note removed: "ADC: 5,6,8-18"
- note removed: "External OPAMP x50 + Internal x2"
- note removed: "No Osc"
- moved on the sheet: C15, C16, C7, C8, C9, R1, R10, SW_BOOT1, SW_BOOT2

Commit message: 10.04.2026
Parts:
- removed U2: AT32F405CCT, Package_QFP:LQFP-48_7x7mm_P0.5mm, symbol Kicad symbols:AT32F405CCT
- removed U8: STM32G473CCTx, Package_QFP:LQFP-48_7x7mm_P0.5mm, symbol MCU_ST_STM32G4:STM32G473CCTx
- removed U9: STM32G473RCTx, Package_QFP:LQFP-64_10x10mm_P0.5mm, symbol MCU_ST_STM32G4:STM32G473RCTx
- added C24, C25: 15pF, symbol Device:C_Small
- added C26: 100nF, Capacitor_SMD:C_0402_1005Metric, symbol Device:C_Small
- added R16, R17, R18, R19: 330R, symbol Device:R_Small
- added U2: STM32G474CBTx, Package_QFP:LQFP-48_7x7mm_P0.5mm, symbol MCU_ST_STM32G4:STM32G474CBTx
- added Y1: 8Mhz 12pF, symbol Device:Crystal_GND24_Small
- R1: value 22k -> 33k
- R4: value 12k 1% -> 330R
Connections:
- net +3.3V: now also U2.1 (VBAT), U2.24 (VDD), U2.36 (VDD), U2.48 (VDD)
- net +3.3VA: now also C26.2, U2.20 (VREF+), U2.21 (VDDA)
- net ADC0: now also U2.8 (PA0)
- net ADC1: now also U2.30 (PA8)
- net BOOT0: now also U2.45 (PB8)
- net D+: now also U2.33 (PA11)
- net D-: now also U2.34 (PA12)
- net DISCHARGE0: now also U2.10 (PA2)
- net DISCHARGE1: now also U2.32 (PA10)
- net GND: now also C24.2, C25.1, C26.1, U2.19 (VSSA), U2.23 (VSS), U2.35 (VSS), U2.47 (VSS), Y1.2, Y1.4; no longer R4.1
- net MUX_EN0: now also U2.12 (PA4)
- net MUX_EN1: now also U2.44 (PB7)
- net RESET: now also U2.7 (PG10)
- net ROW0: now also R4.1
- net ROW1: now also R19.1
- net ROW2: now also R18.1
- net ROW3: now also R17.1
- net ROW4: now also R16.1
- net SWCLK: now also U2.38 (PA14)
- net SWDIO: now also U2.37 (PA13)
- net SWO: now also U2.40 (PB3)
- net at R4.2: now also U2.25 (PB11)
- new net: R16.2, U2.29 (PB15)
- new net: R17.2, U2.28 (PB14)
- new net: C24.1, U2.5 (PF0), Y1.1
- new net: C25.2, U2.6 (PF1), Y1.3
- new net: R18.2, U2.27 (PB13)
- new net: R19.2, U2.26 (PB12)
- new net MUX0_S0: U2.13 (PA5)
- new net MUX0_S1: U2.15 (PA7)
- new net MUX0_S2: U2.14 (PA6)
- new net MUX1_S0: U2.43 (PB6)
- new net MUX1_S1: U2.41 (PB4)
- new net MUX1_S2: U2.42 (PB5)
- no-connect marks 3 -> 6
Other:
- note added: "5 - ADC1 6 - ADC2 8 - ADC12 9 - ADC12 10 - ADC1 11 - ADC1 12 - ADC2 13 - ADC2 14 - ADC2 15 - ADC2 16 - ADC3/ADC1 17 - ADC3/ADC1 18 - ADC2 25 - ADC12 26 - ADC4/ADC1 27 - ADC3 28 - ADC4/ADC1 29 - ADC4/ADC2 30 - ADC5 31 - ADC5"
- note removed: "ADC 10-19"
- note removed: "ST rec: 10n + 1u"
- moved on the sheet: C2, C3, C4, C5, C6, C7, C8, C9

Commit message: 12.04.2026
Parts:
- removed C15: 1uF, Capacitor_SMD:C_0603_1608Metric, symbol Device:C_Small
- removed C26: 100nF, Capacitor_SMD:C_0402_1005Metric, symbol Device:C_Small
- removed J2: Conn_ARM_SWD_TagConnect_TC2030-NL, PCM_marbastlib-various:CON_TC2030_outlined, symbol Connector:Conn_ARM_SWD_TagConnect_TC2030-NL
- removed SW_BOOT1, SW_RST1: SW_Push, TestPoint:TestPoint_2Pads_Pitch2.54mm_Drill0.8mm, symbol Switch:SW_Push
- removed U4: TPS7A2033, Package_TO_SOT_SMD:SOT-23-5, symbol Kicad symbols:TPS7A20xxx SOT-23-5
- added C10, C12: 470pF, Capacitor_SMD:C_0603_1608Metric, symbol Device:C_Small
- added J2: Conn_right, Connector_FFC-FPC:TE_1-84953-6_1x16-1MP_P1.0mm_Horizontal, symbol Connector_Generic:Conn_01x16
- added J3: Conn_left, Connector_FFC-FPC:TE_1-84953-6_1x16-1MP_P1.0mm_Horizontal, symbol Connector_Generic:Conn_01x16
- added J4: SOICbite_connector, Kicad footprints:SOIC_clipProgSmall, symbol Connector_Generic:Conn_02x04_Top_Bottom
- added R3, R6, R7: 330R, Resistor_SMD:R_0603_1608Metric, symbol Device:R_Small
- added U3: TLV75533PDBV, Package_TO_SOT_SMD:SOT-23-5, symbol Regulator_Linear:TLV75533PDBV
- C11: renamed from C25; footprint (none) -> Capacitor_SMD:C_0402_1005Metric
- C15: renamed from C1; footprint (none) -> Capacitor_SMD:C_0402_1005Metric
- C9: renamed from C24; footprint (none) -> Capacitor_SMD:C_0402_1005Metric
- F1: footprint Fuse:Fuse_0603_1608Metric -> Fuse:Fuse_1206_3216Metric
- R1: renamed from R2; footprint Resistor_SMD:R_0402_1005Metric -> Resistor_SMD:R_0603_1608Metric
- R10: renamed from R18; footprint (none) -> Resistor_SMD:R_0603_1608Metric
- R11: renamed from R10; value 22R -> 10R
- R2: renamed from R3; footprint Resistor_SMD:R_0402_1005Metric -> Resistor_SMD:R_0603_1608Metric
- R4: renamed from R17; footprint (none) -> Resistor_SMD:R_0603_1608Metric
- R5: renamed from R16; footprint (none) -> Resistor_SMD:R_0603_1608Metric
- R8: renamed from R4; footprint (none) -> Resistor_SMD:R_0603_1608Metric
- R9: renamed from R19; footprint (none) -> Resistor_SMD:R_0603_1608Metric
- SW_BOOT1: renamed from SW_BOOT2; now fitted; now in the parts list
- SW_RST1: renamed from SW_RST2; now fitted; now in the parts list
- U2: renamed from U1; footprint Package_TO_SOT_SMD:SOT-563 -> Package_TO_SOT_SMD:SOT-23-6
- Y1: footprint (none) -> Crystal:Crystal_SMD_3225-4Pin_3.2x2.5mm
- renumbered C2 to C1, C3 to C2, C4 to C3, C5 to C4, C6 to C5, C7 to C6, C8 to C7, C9 to C8, R1 to R12, U2 to U1
Connections:
- net +3.3V: now also J2.1 (Pin_1), J3.16 (Pin_16), J4.5 (Pin_5), U3.5 (OUT)
- net +5V: now also C13.2, U3.1 (IN), U3.3 (EN); no longer C13.1
- net ADC0: now also J2.3 (Pin_3), R3.2; no longer U1.8 (PA0)
- net ADC1: now also J3.14 (Pin_14), R7.2; no longer U1.30 (PA8)
- net D+: now also U1.34 (PA12); no longer U1.33 (PA11)
- net D-: now also U1.33 (PA11); no longer U1.34 (PA12)
- net DISCHARGE0: now also U1.26 (PB12), J2.5 (Pin_5); no longer U1.10 (PA2)
- net DISCHARGE1: now also U1.22 (PB10), J3.12 (Pin_12); no longer U1.32 (PA10)
- net GND: now also C13.1, C10.2, C12.2, J2.2 (Pin_2), J2.4 (Pin_4), J3.13 (Pin_13), J3.15 (Pin_15), J4.1 (Pin_1), U3.2 (GND); no longer C13.2
- net MUX0_S0: now also U1.41 (PB4), J2.9 (Pin_9); no longer U1.13 (PA5)
- net MUX0_S1: now also U1.42 (PB5), J2.8 (Pin_8); no longer U1.15 (PA7)
- net MUX0_S2: now also U1.43 (PB6), J2.7 (Pin_7); no longer U1.14 (PA6)
- net MUX1_S0: now also U1.14 (PA6), J3.8 (Pin_8); no longer U1.43 (PB6)
- net MUX1_S1: now also U1.15 (PA7), J3.9 (Pin_9); no longer U1.41 (PB4)
- net MUX1_S2: now also U1.16 (PB0), J3.10 (Pin_10); no longer U1.42 (PB5)
- net RESET: now also J4.8 (Pin_8)
- net ROW0: now also J2.11 (Pin_11), J3.6 (Pin_6)
- net ROW1: now also J2.12 (Pin_12), J3.5 (Pin_5)
- net ROW2: now also J2.13 (Pin_13), J3.4 (Pin_4)
- net ROW3: now also J2.14 (Pin_14), J3.3 (Pin_3)
- net ROW4: now also J2.15 (Pin_15), J3.2 (Pin_2)
- net SWCLK: now also J4.3 (Pin_3)
- net SWDIO: now also J4.4 (Pin_4)
- net SWO: now also J4.2 (Pin_2)
- net at R5.2: now also U1.31 (PA9); no longer U1.29 (PB15)
- net at R4.2: now also U1.30 (PA8); no longer U1.28 (PB14)
- net at R8.2: now also U1.27 (PB13); no longer U1.25 (PB11)
- net at R10.2: now also U1.29 (PB15); no longer U1.27 (PB13)
- net at R9.2: now also U1.28 (PB14); no longer U1.26 (PB12)
- net at U1.11 (PA3): now also C10.1, R3.1
- net MUX1_S3: now reaches U1.17 (PB1)
- net MUX1_S3: now also J3.11 (Pin_11)
- net at U1.18 (PB2): now also C12.1, R7.1
- net MUX0_EN: now reaches U1.39 (PA15)
- net MUX0_EN: now also J2.10 (Pin_10)
- net MUX_EN0: no longer names the net of U1.12 (PA4)
- net MUX_EN1 renamed MUX0_S3
- net MUX0_S3: now also J2.6 (Pin_6)
- new net: R6.2, U1.32 (PA10)
- new net MUX1_EN: J3.7 (Pin_7), U1.13 (PA5)
- new net ROW5: J2.16 (Pin_16), J3.1 (Pin_1), R6.1
- no-connect marks 6 -> 12
Other:
- removed sheet Delta MATRIX
- removed sheet Delta MUX
- note added: "Универсальная плата до 100% qfp-48 -> MUX 16ch x2 qfp-64 -> MUX 16ch x3+ MUX и OPAMP вместе на дочерней плате"
- moved on the sheet: C1, C11, C15, C16, C2, C3, C4, C5, C6, C7, C8, C9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
