File: Libra mini EC MATRIX.kicad_sch (KiCad schematic)
At the start: 65 parts, among them SW1 EC_SW, SW10 EC_SW, SW11 EC_SW, SW12 EC_SW, SW13 EC_SW, SW14 EC_SW, SW15 EC_SW, SW16 EC_SW, SW17 EC_SW, SW18 EC_SW, SW19 EC_SW, SW2 EC_SW, SW20 EC_SW, SW21 EC_SW, SW22 EC_SW, SW23 EC_SW, SW24 EC_SW, SW25 EC_SW, SW26 EC_SW, SW27 EC_SW, SW28 EC_SW, SW29 EC_SW, SW3 EC_SW, SW30 EC_SW, SW31 EC_SW, SW32 EC_SW, SW33 EC_SW, SW34 EC_SW, SW35 EC_SW, SW36 EC_SW, SW37 EC_SW, SW38 EC_SW, SW39 EC_SW, SW4 EC_SW, SW40 EC_SW, SW41 EC_SW, SW42 EC_SW, SW43 EC_SW, SW44 EC_SW, SW45 EC_SW, SW46 EC_SW, SW47 EC_SW, SW48 EC_SW, SW49 EC_SW, SW5 EC_SW, SW50 EC_SW, SW6 EC_SW, SW7 EC_SW, SW8 EC_SW, SW9 EC_SW

Commit message: 14.04.2026
Parts:
- added S51: MX_stab, PCM_marbastlib-mx:STAB_MX_2.25u, symbol PCM_marbastlib-mx:MX_stab
- added S52: MX_stab, PCM_marbastlib-mx:STAB_MX_2u, symbol PCM_marbastlib-mx:MX_stab
- added SW51, SW52, SW53: EC_SW, Kicad footprints:ecs_pad_hybrid_hotswap_1.25-1_libra_2.381, symbol Kicad symbols:EC_SW
- added SW54, SW55: EC_SW, Kicad footprints:ecs_pad_hybrid_hotswap_1.810, symbol Kicad symbols:EC_SW
- SW39, SW40, SW50: footprint Kicad footprints:ecs_pad_1U_hybrid_hotswap_V2 -> Kicad footprints:ecs_pad_hybrid_hotswap_1.25-1_libra_2.381
- SW41, SW42, SW43, SW44, SW49: now not fitted; now left out of the parts list
- SW45: footprint Kicad footprints:ecs_pad_hybrid_hotswap_1.25-1_libra_7.239 -> Kicad footprints:ecs_pad_1U_hybrid_hotswap_V2; now not fitted; now left out of the parts list
- SW46: footprint Kicad footprints:ecs_pad_hybrid_hotswap_1.25-1_libra_2.381 -> Kicad footprints:ecs_pad_1U_hybrid_hotswap_V2; now not fitted; now left out of the parts list
- SW48: footprint Kicad footprints:ecs_pad_hybrid hotswap_1.25-1_libra_2.286 -> Kicad footprints:ecs_pad_1U_hybrid_hotswap_V2; now not fitted; now left out of the parts list
Connections:
- net COL0: now also SW48.1
- net COL1: now also SW49.1
- net COL3: now also SW50.1
- net COL4: now also SW51.1
- net COL6: now also SW52.1
- net COL7: now also SW53.1; no longer SW48.1
- net COL8: now also SW54.1; no longer SW49.1
- net COL9: now also SW55.1; no longer SW50.1
- net GND: now also SW50.3 (SG), SW51.3 (SG), SW52.3 (SG), SW53.3 (SG), SW54.3 (SG), SW55.3 (SG)
- net ROW3: now also SW51.2, SW52.2, SW53.2, SW54.2, SW55.2
Other:
- moved on the sheet: D1, D10, D11, D12, D2, D3, D4, D5, D6, D7, D8, D9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
