File: Libra mini EC.kicad_sch (KiCad schematic)
At the start: 40 parts, among them J1 USB_C_Receptacle_USB2.0_16P, J2 Analog joystick 5 pin, J3 Conn_01x18, J4 Conn_01x18, U1 STM32G474CBTx, U2 USBLC6-2SC6, U3 TPS7A2033, U4 TPS7A2033, U5 TPS7A2033, Y1 8Mhz 12pF

Commit message: 13.04.2026
Parts:
- added C11, C12, C13, C14: 220pF, Capacitor_SMD:C_0603_1608Metric, symbol Device:C_Small
- added R3, R4, R5, R6: 330R, Resistor_SMD:R_0603_1608Metric, symbol Device:R_Small
- renumbered C11 to C15, C12 to C16, C13 to C17, C14 to C18, C15 to C19, C16 to C20, C17 to C21, C18 to C22, C19 to C23, R6 to R10, R7 to R11, R8 to R12, R3 to R7, R4 to R8, R5 to R9
Connections:
- net ADC0_IN: now also R3.2; no longer U1.14 (PA6)
- net ADC1_IN: now also R4.2; no longer U1.15 (PA7)
- net ADC2_IN: now also R5.2; no longer U1.30 (PA8)
- net ADC3_IN: now also R6.2; no longer U1.31 (PA9)
- net GND: now also C11.2, C12.2, C13.2, C14.2
- new net: C14.1, R6.1, U1.31 (PA9)
- new net: C13.1, R5.1, U1.30 (PA8)
- new net: C11.1, R3.1, U1.14 (PA6)
- new net: C12.1, R4.1, U1.15 (PA7)
Other:
- moved on the sheet: J2
