File: Libra mini EC.kicad_sch (KiCad schematic)
At the start: 48 parts, among them J1 USB_C_Receptacle_USB2.0_16P, J2 Conn_01x08, J3 Conn_01x18, J4 Conn_01x18, U1 STM32G474CBTx, U2 USBLC6-2SC6, U3 TPS7A2033, U4 TPS7A2033, U5 TPS7A2033, Y1 8Mhz 12pF

Commit message: 14.04.2026
Connections:
- net +5V: now also J4.17 (Pin_17); no longer J4.2 (Pin_2)
- net ADC2_IN: now also J4.10 (Pin_10); no longer J4.9 (Pin_9)
- net ADC3_IN: now also J4.14 (Pin_14); no longer J4.5 (Pin_5)
- net DISCHARGE2: now also J4.12 (Pin_12); no longer J4.7 (Pin_7)
- net DISCHARGE3: now also J4.16 (Pin_16); no longer J4.3 (Pin_3)
- net GND: now also J4.11 (Pin_11), J4.13 (Pin_13), J4.15 (Pin_15), J4.9 (Pin_9); no longer J4.10 (Pin_10), J4.4 (Pin_4), J4.6 (Pin_6), J4.8 (Pin_8)
- net MUX1_EN: now also J4.6 (Pin_6); no longer J4.13 (Pin_13)
- net MUX_S0: now also J4.8 (Pin_8); no longer J4.11 (Pin_11)
- net MUX_S1: now also J4.7 (Pin_7); no longer J4.12 (Pin_12)
- net RGB: now also J4.1 (Pin_1); no longer J4.18 (Pin_18)
- net RGB_START: now also J4.18 (Pin_18); no longer J4.1 (Pin_1)
- net ROW0: now also J4.2 (Pin_2); no longer J4.17 (Pin_17)
- net ROW1: now also J4.3 (Pin_3); no longer J4.16 (Pin_16)
- net ROW2: now also J4.4 (Pin_4); no longer J4.15 (Pin_15)
- net ROW3: now also J4.5 (Pin_5); no longer J4.14 (Pin_14)
Changed lines of the file:
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@@
 	(symbol
 		(lib_id "Connector_Generic:Conn_01x18")
-		(at 162.56 172.72 0)
+		(at 162.56 175.26 0)
+		(mirror x)
 		(unit 1)
 		(exclude_from_sim no)
@@
 		(on_board yes)
 		(dnp no)
-		(fields_autoplaced yes)
 		(property "Reference" "J4"
-			(at 165.1 172.7199 0)
+			(at 165.1 175.2601 0)
 			(effects
 				(font
@@
 		)
 		(property "Value" "Conn_01x18"
-			(at 165.1 175.2599 0)
+			(at 165.1 172.7201 0)
 			(effects
 				(font
@@
 		)
 		(property "Footprint" "Connector_FFC-FPC:JUSHUO_AFA07-S18FCA-00_1x18-1MP_P1.0mm_Horizontal"
-			(at 162.56 172.72 0)
+			(at 162.56 175.26 0)
 			(effects
 				(font
@@
 		)
 		(property "Datasheet" "~"
-			(at 162.56 172.72 0)
+			(at 162.56 175.26 0)
 			(effects
 				(font
@@
 		)
 		(property "Description" "Generic connector, single row, 01x18, script generated (kicad-library-utils/schlib/autogen/connector/)"
-			(at 162.56 172.72 0)
+			(at 162.56 175.26 0)
 			(effects
 				(font
