File: Libra mini EC.kicad_sch (KiCad schematic)
At the start: 42 parts, among them J1 USB_C_Receptacle_USB2.0_16P, J2 Conn_01x08, J3 Conn_01x18, J4 Conn_01x18, U1 STM32G474CBTx, U2 USBLC6-2SC6, U3 TPS7A2033, Y1 8Mhz 12pF

Commit message: 16.04.2026
Connections:
- net MUX0_EN: now also U1.43 (PB6); no longer U1.42 (PB5)
- net MUX1_EN: now also U1.44 (PB7); no longer U1.43 (PB6)
- net MUX_S0: now also U1.41 (PB4); no longer U1.40 (PB3)
- net MUX_S1: now also U1.42 (PB5); no longer U1.41 (PB4)
- net SWCLK: now also U1.38 (PA14)
- net SWDIO: now also U1.37 (PA13)
- net SWO: now also U1.40 (PB3)
