File: Libra mini EC.kicad_pcb (KiCad board)
At the start: 2 copper layers, 273.8 x 207.5 mm, 149 parts, among them J1 USB_C_Receptacle_USB2.0_16P, J2 Conn_01x08, J3 Conn_01x18, J4 Conn_01x18, SW1 EC_SW, SW10 EC_SW, SW11 EC_SW, SW12 EC_SW, SW13 EC_SW, SW14 EC_SW, SW15 EC_SW, SW16 EC_SW, SW17 EC_SW, SW18 EC_SW, SW19 EC_SW, SW2 EC_SW, SW20 EC_SW, SW21 EC_SW, SW22 EC_SW, SW23 EC_SW, SW24 EC_SW, SW25 EC_SW, SW26 EC_SW, SW27 EC_SW, SW28 EC_SW, SW29 EC_SW, SW3 EC_SW, SW30 EC_SW, SW31 EC_SW, SW32 EC_SW, SW33 EC_SW, SW34 EC_SW, SW35 EC_SW, SW36 EC_SW, SW37 EC_SW, SW38 EC_SW, SW39 EC_SW, SW4 EC_SW, SW40 EC_SW, SW41 EC_SW, SW42 EC_SW, SW43 EC_SW, SW44 EC_SW, SW45 EC_SW, SW46 EC_SW, SW47 EC_SW, SW48 EC_SW, SW49 EC_SW, SW5 EC_SW, SW50 EC_SW, SW6 EC_SW, SW7 EC_SW, SW8 EC_SW, SW9 EC_SW, U1 STM32G474CBTx, U2 USBLC6-2SC6, U3 TPS7A2033, U4 TPS7A2033, U5 TPS7A2033, U6 OPA2365, U7 4052, U8 OPA2365, U9 4052, Y1 8Mhz 12pF

Commit message: 14.04.2026
Parts:
- removed REF** (x4): MountingHole_2.2mm_M2_DIN965_Pad, MountingHole:MountingHole_2.2mm_M2_DIN965_Pad
- removed SW41, SW42, SW43, SW44, SW49: EC_SW, Kicad footprints:ecs_pad_1U_hybrid_hotswap_V2
- removed SW45: EC_SW, Kicad footprints:ecs_pad_hybrid_hotswap_1.25-1_libra_7.239
- removed SW46: EC_SW, Kicad footprints:ecs_pad_hybrid_hotswap_1.25-1_libra_2.381
- removed SW48: EC_SW, Kicad footprints:ecs_pad_hybrid hotswap_1.25-1_libra_2.286
- added S51: MX_stab, PCM_marbastlib-mx:STAB_MX_2.25u, F.Cu at (112.2, 87.1)
- added S52: MX_stab, PCM_marbastlib-mx:STAB_MX_2u, F.Cu at (167.5, 87.3)
- added SW51: EC_SW, Kicad footprints:ecs_pad_hybrid_hotswap_1.25-1_libra_2.381, F.Cu at (112.2, 87.1)
- added SW52: EC_SW, Kicad footprints:ecs_pad_hybrid_hotswap_1.25-1_libra_2.381, F.Cu at (167.5, 87.3)
- added SW53: EC_SW, Kicad footprints:ecs_pad_hybrid_hotswap_1.25-1_libra_2.381, F.Cu at (200.6, 82.7)
- added SW54: EC_SW, Kicad footprints:ecs_pad_hybrid_hotswap_1.810, F.Cu at (244.7, 79.5)
- added SW55: EC_SW, Kicad footprints:ecs_pad_hybrid_hotswap_1.810, F.Cu at (268.5, 79.5)
- SW39, SW40, SW50: footprint Kicad footprints:ecs_pad_1U_hybrid_hotswap_V2 -> Kicad footprints:ecs_pad_hybrid_hotswap_1.25-1_libra_2.381
- moved SW50 183.0 mm to (81.6, 82.8), turned to -8 degrees
- moved J3 127.1 mm to (259.0, 144.2)
- moved J4 127.1 mm to (276.6, 143.5)
- moved J1 127.1 mm to (267.8, 96.0)
- moved U1 127.1 mm to (267.8, 111.1)
- moved C24 14.2 mm to (356.7, 83.3)
- moved SW10 5.45 mm to (211.5, 23.4)
- moved SW7 5.45 mm to (154.9, 31.4)
- moved SW8 5.45 mm to (173.7, 28.7)
- moved SW9 5.45 mm to (192.6, 26.1)
- moved SW12 5.16 mm to (250.4, 21.8)
- moved SW13 5.16 mm to (269.5, 21.8)
- moved SW11 5.16 mm to (231.4, 21.8)
- moved S47 5.16 mm to (260.0, 21.8)
- moved SW47 5.16 mm to (260.0, 21.8)
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Connections:
- J4 pad 1: RGB_START -> RGB
- J4 pad 10: GND -> ADC2_IN
- J4 pad 11: MUX_S0 -> GND
- J4 pad 12: MUX_S1 -> DISCHARGE2
- J4 pad 13: MUX1_EN -> GND
- J4 pad 14: ROW3 -> ADC3_IN
- J4 pad 15: ROW2 -> GND
- J4 pad 16: ROW1 -> DISCHARGE3
- J4 pad 17: ROW0 -> +5V
- J4 pad 18: RGB -> RGB_START
- J4 pad 2: +5V -> ROW0
- J4 pad 3: DISCHARGE3 -> ROW1
- J4 pad 4: GND -> ROW2
- J4 pad 5: ADC3_IN -> ROW3
- J4 pad 6: GND -> MUX1_EN
- J4 pad 7: DISCHARGE2 -> MUX_S1
- J4 pad 8: GND -> MUX_S0
- J4 pad 9: ADC2_IN -> GND
- SW50 pad 1: COL9 -> COL3
- SW50 pad 3: unconnected-(SW50-SG-Pad3) -> GND
Other:
- board size 273.8 x 207.5 mm -> 269.5 x 183.8 mm
