File: Delta EC.kicad_sch (KiCad schematic)
At the start: 43 parts, among them J1 USB_C_Receptacle_USB2.0_16P, J2 SOICbite, J3 FFC Daughter side, J4 FFC Main side, J5 JSB USB, U1 STM32G474CBTx, U2 USBLC6-2SC6, U3 TPS7A2033, Y1 8Mhz 12pF

Commit message: 17.04.2026
Parts:
- J3, J4: footprint Connector_FFC-FPC:Amphenol_F32Q-1A7x1-11018_1x18-1MP_P0.5mm_Horizontal -> Connector_FFC-FPC:TE_1-1734839-8_1x18-1MP_P0.5mm_Horizontal
Changed lines of the file:
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@@
 			)
 		)
-		(property "Footprint" "Connector_FFC-FPC:Amphenol_F32Q-1A7x1-11018_1x18-1MP_P0.5mm_Horizontal"
+		(property "Footprint" "Connector_FFC-FPC:TE_1-1734839-8_1x18-1MP_P0.5mm_Horizontal"
 			(at 106.68 172.72 0)
 			(effects
@@
 			)
 		)
-		(property "Footprint" "Connector_FFC-FPC:Amphenol_F32Q-1A7x1-11018_1x18-1MP_P0.5mm_Horizontal"
+		(property "Footprint" "Connector_FFC-FPC:TE_1-1734839-8_1x18-1MP_P0.5mm_Horizontal"
 			(at 162.56 172.72 0)
 			(effects
