File: Delta EC.kicad_pcb (KiCad board)
At the start: 2 copper layers, 301.7 x 106 mm, 139 parts, among them J1 USB_C_Receptacle_USB2.0_16P, J2 SOICbite, J3 FFC Daughter side, J4 FFC Main side, J5 JSB USB, SW1 EC_SW, SW10 EC_SW, SW11 EC_SW, SW12 EC_SW, SW13 EC_SW, SW14 EC_SW, SW15 EC_SW, SW16 EC_SW, SW17 EC_SW, SW18 EC_SW, SW19 EC_SW, SW2 EC_SW, SW20 EC_SW, SW21 EC_SW, SW22 EC_SW, SW23 EC_SW, SW24 EC_SW, SW25 EC_SW, SW26 EC_SW, SW27 EC_SW, SW28 EC_SW, SW29 EC_SW, SW3 EC_SW, SW30 EC_SW, SW31 EC_SW, SW32 EC_SW, SW33 EC_SW, SW34 EC_SW, SW35 EC_SW, SW36 EC_SW, SW37 EC_SW, SW38 EC_SW, SW39 EC_SW, SW4 EC_SW, SW40 EC_SW, SW47 EC_SW, SW5 EC_SW, SW50 EC_SW, SW51 EC_SW, SW52 EC_SW, SW53 EC_SW, SW54 EC_SW, SW55 EC_SW, SW6 EC_SW, SW7 EC_SW, SW8 EC_SW, SW9 EC_SW, U1 STM32G474CBTx, U2 USBLC6-2SC6, U3 TPS7A2033, U6 OPA2365, U7 4052, U8 OPA2365, U9 4052, Y1 8Mhz 12pF

Commit message: 17.04.2026
Parts:
- J3, J4: footprint Connector_FFC-FPC:Amphenol_F32Q-1A7x1-11018_1x18-1MP_P0.5mm_Horizontal -> Connector_FFC-FPC:TE_1-1734839-8_1x18-1MP_P0.5mm_Horizontal
- moved J3 81.7 mm to (148.4, 52.0), turned to 90 degrees
- moved J4 68.4 mm to (133.0, 52.0)
- moved D5 26.4 mm to (70.1, 85.6)
- moved R19 14.4 mm to (66.3, 72.2), turned to 0 degrees
- moved R18 11.5 mm to (63.1, 72.2)
- moved R13 5.16 mm to (63.5, 81.8)
- moved R14 4.77 mm to (60.3, 81.8), turned to 0 degrees
- moved D6 3.57 mm to (118.7, 77.4)
- moved D2 1.98 mm to (70.2, 31.0)
- moved C26 1.86 mm to (65.9, 74.2), turned to -90 degrees
- moved C24 1.05 mm to (54.4, 66.3), turned to 180 degrees
- moved U7 0.32 mm to (57.5, 69.8)
- moved U6 0.12 mm to (62.3, 77.0)
Connections:
- R15 pad 1: COL4 -> COL5
- R20 pad 1: COL5 -> COL4
- U7 pad 2: COL5 -> COL4
- U7 pad 5: COL4 -> COL5
Routing:
- net COL7: track 68.0 -> 0.00 mm
- net COL6: track 61.2 -> 0.00 mm
- net COL11: track 59.9 -> 0.00 mm
- net COL10: track 46.9 -> 0.00 mm
- net COL9: track 38.7 -> 0.00 mm
- net COL8: track 38.7 -> 0.00 mm
- net COL5: track 45.0 -> 67.6 mm
- net ROW0: track 0.00 -> 18.3 mm
- net COL4: track 64.8 -> 48.9 mm
- net ADC1_IN: track 0.00 -> 8.58 mm
- net Net-(U6B--): track 0.00 -> 7.63 mm
- net ADC0_IN: track 0.00 -> 6.99 mm
- net COL0: track 42.7 -> 48.0 mm
- net +3.3VA: track 4.32 -> 9.53 mm, vias 0 -> 2
- net Net-(U6A--): track 0.00 -> 3.92 mm
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Other:
- outline, holes or cut-outs redrawn

Commit message: 12.05.2026
Parts:
- SW1, SW10, SW11, SW12, SW13, SW14, SW15, SW16, SW17, SW18, SW19, SW2, SW20, SW21, SW22, SW23, SW24, SW26, SW27, SW28, SW29, SW3, SW30, SW31, SW37, SW38, SW4, SW47, SW5, SW6, SW7, SW8, SW9: footprint Kicad footprints:ecs_pad_1U_hybrid_hotswap_V2 -> Kicad footprints:ecs_pad_1U_hybrid_hotswap_V3
- SW25, SW32, SW33, SW34, SW35, SW36: footprint Kicad footprints:ecs_pad_1U_hybrid_hotswap_V2_switched_sides -> Kicad footprints:ecs_pad_1U_hybrid_hotswap_V3_switched_sides
- SW39, SW40, SW50, SW51, SW52, SW53, SW54, SW55: footprint Kicad footprints:ecs_pad_hybrid_hotswap_2.381_V2 -> Kicad footprints:ecs_pad_hybrid_hotswap_2.381_V3
